File: hardware/yeg-channel/adc.kicad_sch (KiCad schematic)
At the start: 23 parts, among them U10 HX71708, U11 74HC4051, U7 HX71708, U8 HX71708, U9 HX71708

Commit message: fixes and add pcb layout
Parts:
- removed C50: 100n, Capacitor_SMD:C_0603_1608Metric, symbol Device:C_Small
- removed R13, R15: 200, Resistor_SMD:R_0603_1608Metric, symbol Device:R_Small
- renumbered R14 to R13
Connections:
- net CINA+ is gone; now on net SRB2: R12.1
Other:
- title: Yet Another EXG Channel Board -> YEG Channel Board
Changed lines of the file:
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@@
   (paper "A4")
   (title_block
-    (title "Yet Another EXG Channel Board")
+    (title "YEG Channel Board")
     (date "2024-02-07")
     (rev "1")
@@
   (junction (at 140.97 105.41) (diameter 0) (color 0 0 0 0)
   )
-  (junction (at 133.35 163.83) (diameter 0) (color 0 0 0 0)
-  )
   (junction (at 77.47 52.07) (diameter 0) (color 0 0 0 0)
   )
@@
   )
   (junction (at 54.61 34.29) (diameter 0) (color 0 0 0 0)
-  )
-  (junction (at 133.35 156.21) (diameter 0) (color 0 0 0 0)
   )
   (junction (at 140.97 54.61) (diameter 0) (color 0 0 0 0)
@@
     (stroke (width 0) (type default))
   )
-  (wire (pts (xy 127 156.21) (xy 133.35 156.21))
-    (stroke (width 0) (type default))
-  )
   (wire (pts (xy 140.97 111.76) (xy 140.97 113.03))
     (stroke (width 0) (type default))
@@
     (stroke (width 0) (type default))
   )
-  (wire (pts (xy 119.38 163.83) (xy 121.92 163.83))
-    (stroke (width 0) (type default))
-  )
   (wire (pts (xy 31.75 149.86) (xy 31.75 142.24))
     (stroke (width 0) (type default))
@@
     (stroke (width 0) (type default))
   )
-  (wire (pts (xy 119.38 156.21) (xy 121.92 156.21))
-    (stroke (width 0) (type default))
-  )
   (wire (pts (xy 50.8 154.94) (xy 53.34 154.94))
     (stroke (width 0) (type default))
@@
     (stroke (width 0) (type default))
   )
-  (wire (pts (xy 133.35 162.56) (xy 133.35 163.83))
-    (stroke (width 0) (type default))
-  )
   (wire (pts (xy 43.18 172.72) (xy 43.18 175.26))
     (stroke (width 0) (type default))
@@
     (stroke (width 0) (type default))
   )
-  (wire (pts (xy 133.35 163.83) (xy 143.51 163.83))
-    (stroke (width 0) (type default))
-  )
   (wire (pts (xy 100.33 46.99) (xy 104.14 46.99))
     (stroke (width 0) (type default))
@@
     (stroke (width 0) (type default))
   )
-  (wire (pts (xy 133.35 156.21) (xy 143.51 156.21))
-    (stroke (width 0) (type default))
-  )
   (wire (pts (xy 44.45 82.55) (xy 44.45 90.17))
     (stroke (width 0) (type default))
   )
-  (wire (pts (xy 127 163.83) (xy 133.35 163.83))
-    (stroke (width 0) (type default))
-  )
   (wire (pts (xy 132.08 52.07) (xy 149.86 52.07))
     (stroke (width 0) (type default))
@@
   )
   (wire (pts (xy 68.58 111.76) (xy 68.58 113.03))
-    (stroke (width 0) (type default))
-  )
-  (wire (pts (xy 133.35 156.21) (xy 133.35 157.48))
     (stroke (width 0) (type default))
   )
@@
     (effects (font (size 1.27 1.27)) (justify left bottom))
   )
-  (label "IN+" (at 143.51 156.21 0) (fields_autoplaced)
-    (effects (font (size 1.27 1.27)) (justify left bottom))
-  )
   (label "IN+" (at 104.14 156.21 0) (fields_autoplaced)
     (effects (font (size 1.27 1.27)) (justify left bottom))
@@
     (effects (font (size 1.27 1.27)) (justify left bottom))
   )
-  (label "IN-" (at 143.51 163.83 0) (fields_autoplaced)
-    (effects (font (size 1.27 1.27)) (justify left bottom))
-  )
   (label "PD_SCK2" (at 85.09 102.87 0) (fields_autoplaced)
     (effects (font (size 1.27 1.27)) (justify left bottom))
@@
     (effects (font (size 1.27 1.27)) (justify right))
   )
-  (hierarchical_label "CINA+" (shape passive) (at 80.01 156.21 180) (fields_autoplaced)
+  (hierarchical_label "SRB2" (shape passive) (at 80.01 156.21 180) (fields_autoplaced)
     (effects (font (size 1.27 1.27)) (justify right))
   )
@@
     (effects (font (size 1.27 1.27)) (justify right))
   )
-  (hierarchical_label "SRB1" (shape passive) (at 119.38 163.83 180) (fields_autoplaced)
-    (effects (font (size 1.27 1.27)) (justify right))
-  )
   (hierarchical_label "CS0" (shape input) (at 31.75 154.94 180) (fields_autoplaced)
     (effects (font (size 1.27 1.27)) (justify right))
@@
     (effects (font (size 1.27 1.27)) (justify left))
   )
-  (hierarchical_label "SRB2" (shape passive) (at 119.38 156.21 180) (fields_autoplaced)
-    (effects (font (size 1.27 1.27)) (justify right))
-  )
   (hierarchical_label "CINA-" (shape passive) (at 80.01 163.83 180) (fields_autoplaced)
     (effects (font (size 1.27 1.27)) (justify right))
@@
         (path "/edce6e4b-dbee-4006-90c7-70e47f82b9ee/f9667ef1-4e46-41e1-a5e4-f6ce5d2d23c2"
           (reference "R6") (unit 1)
-        )
-      )
-    )
-  )
-  (symbol (lib_id "Device:C_Small") (at 133.35 160.02 0) (unit 1)
-    (in_bom yes) (on_board yes) (dnp no) (fields_autoplaced)
-    (property "Reference" "C50" (at 135.89 158.7563 0)
-      (effects (font (size 1.27 1.27)) (justify left))
-    )
-    (property "Value" "100n" (at 135.89 161.2963 0)
-      (effects (font (size 1.27 1.27)) (justify left))
-    )
-    (property "Footprint" "Capacitor_SMD:C_0603_1608Metric" (at 133.35 160.02 0)
-      (effects (font (size 1.27 1.27)) hide)
-    )
-    (property "Datasheet" "~" (at 133.35 160.02 0)
-      (effects (font (size 1.27 1.27)) hide)
-    )
-    (property "LCSC ID" "C14663" (at 133.35 160.02 0)
-      (effects (font (size 1.27 1.27)) hide)
-    )
-    (pin "1")
-    (pin "2")
-    (instances
-      (project "yeg-channel"
-        (path "/edce6e4b-dbee-4006-90c7-70e47f82b9ee/f9667ef1-4e46-41e1-a5e4-f6ce5d2d23c2"
-          (reference "C50") (unit 1)
         )
       )
@@
   (symbol (lib_id "Device:R_Small") (at 85.09 163.83 90) (mirror x) (unit 1)
     (in_bom yes) (on_board yes) (dnp no)
-    (property "Reference" "R14" (at 85.09 168.91 90)
+    (property "Reference" "R13" (at 85.09 168.91 90)
       (effects (font (size 1.27 1.27)))
     )
@@
       (project "yeg-channel"
         (path "/edce6e4b-dbee-4006-90c7-70e47f82b9ee/f9667ef1-4e46-41e1-a5e4-f6ce5d2d23c2"
-          (reference "R14") (unit 1)
+          (reference "R13") (unit 1)
         )
       )
@@
         (path "/edce6e4b-dbee-4006-90c7-70e47f82b9ee/f9667ef1-4e46-41e1-a5e4-f6ce5d2d23c2"
           (reference "#PWR055") (unit 1)
-        )
-      )
-    )
-  )
-  (symbol (lib_id "Device:R_Small") (at 124.46 156.21 90) (unit 1)
-    (in_bom yes) (on_board yes) (dnp no) (fields_autoplaced)
-    (property "Reference" "R13" (at 124.46 151.13 90)
-      (effects (font (size 1.27 1.27)))
-    )
-    (property "Value" "200" (at 124.46 153.67 90)
-      (effects (font (size 1.27 1.27)))
-    )
-    (property "Footprint" "Resistor_SMD:R_0603_1608Metric" (at 124.46 156.21 0)
-      (effects (font (size 1.27 1.27)) hide)
-    )
-    (property "Datasheet" "~" (at 124.46 156.21 0)
-      (effects (font (size 1.27 1.27)) hide)
-    )
-    (property "LCSC ID" "C8218" (at 124.46 156.21 0)
-      (effects (font (size 1.27 1.27)) hide)
-    )
-    (pin "1")
-    (pin "2")
-    (instances
-      (project "yeg-channel"
-        (path "/edce6e4b-dbee-4006-90c7-70e47f82b9ee/f9667ef1-4e46-41e1-a5e4-f6ce5d2d23c2"
-          (reference "R13") (unit 1)
         )
       )
@@
         )
       )
-    )
-  )
-  (symbol (lib_id "Device:R_Small") (at 124.46 163.83 90) (mirror x) (unit 1)
-    (in_bom yes) (on_board yes) (dnp no)
-    (property "Reference" "R15" (at 124.46 168.91 90)
-      (effects (font (size 1.27 1.27)))
-    )
-    (property "Value" "200" (at 124.46 166.37 90)
-      (effects (font (size 1.27 1.27)))
-    )
-    (property "Footprint" "Resistor_SMD:R_0603_1608Metric" (at 124.46 163.83 0)
-      (effects (font (size 1.27 1.27)) hide)
-    )
-    (property "Datasheet" "~" (at 124.46 163.83 0)
-      (effects (font (size 1.27 1.27)) hide)
-    )
-    (property "LCSC ID" "C8218" (at 124.46 163.83 0)
-      (effects (font (size 1.27 1.27)) hide)
-    )
-    (pin "1")
-    (pin "2")
-    (instances
-      (project "yeg-channel"
-        (path "/edce6e4b-dbee-4006-90c7-70e47f82b9ee/f9667ef1-4e46-41e1-a5e4-f6ce5d2d23c2"
-          (reference "R15") (unit 1)
-        )
-      )
