File: hardware/yeg-channel/power.kicad_sch (KiCad schematic)
At the start: 51 parts, among them U1 AMS1117-3.3, U2 AMS1117-2.5, U3 LM2664M6X, U4 LM337L_SO8

Commit message: fixes and add pcb layout
Parts:
- added C50: 100n, Capacitor_SMD:C_0603_1608Metric, symbol Device:C_Small
Connections:
- net +3V3: now also C50.1
- net GND: now also C50.2
Other:
- title: Yet Another EXG Channel Board -> YEG Channel Board
Changed lines of the file:
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@@
   (paper "A4")
   (title_block
-    (title "Yet Another EXG Channel Board")
+    (title "YEG Channel Board")
     (date "2024-02-07")
     (rev "1")
@@
   (junction (at 25.4 130.81) (diameter 0) (color 0 0 0 0)
   )
+  (junction (at 45.72 96.52) (diameter 0) (color 0 0 0 0)
+  )
   (junction (at 100.33 25.4) (diameter 0) (color 0 0 0 0)
   )
@@
   (junction (at 25.4 25.4) (diameter 0) (color 0 0 0 0)
   )
+  (junction (at 45.72 88.9) (diameter 0) (color 0 0 0 0)
+  )
   (junction (at 128.27 46.99) (diameter 0) (color 0 0 0 0)
   )
@@
     (stroke (width 0) (type default))
   )
+  (wire (pts (xy 55.88 90.17) (xy 55.88 88.9))
+    (stroke (width 0) (type default))
+  )
   (wire (pts (xy 33.02 62.23) (xy 33.02 57.15))
     (stroke (width 0) (type default))
@@
     (stroke (width 0) (type default))
   )
+  (wire (pts (xy 55.88 88.9) (xy 45.72 88.9))
+    (stroke (width 0) (type default))
+  )
   (wire (pts (xy 76.2 130.81) (xy 86.36 130.81))
     (stroke (width 0) (type default))
@@
     (stroke (width 0) (type default))
   )
+  (wire (pts (xy 55.88 96.52) (xy 45.72 96.52))
+    (stroke (width 0) (type default))
+  )
   (wire (pts (xy 55.88 137.16) (xy 55.88 138.43))
     (stroke (width 0) (type default))
@@
   )
   (wire (pts (xy 121.92 135.89) (xy 121.92 137.16))
+    (stroke (width 0) (type default))
+  )
+  (wire (pts (xy 55.88 95.25) (xy 55.88 96.52))
     (stroke (width 0) (type default))
   )
@@
         )
       )
+    )
+  )
+  (symbol (lib_id "Device:C_Small") (at 55.88 92.71 0) (unit 1)
+    (in_bom yes) (on_board yes) (dnp no) (fields_autoplaced)
+    (property "Reference" "C50" (at 58.42 91.4463 0)
+      (effects (font (size 1.27 1.27)) (justify left))
+    )
+    (property "Value" "100n" (at 58.42 93.9863 0)
+      (effects (font (size 1.27 1.27)) (justify left))
+    )
+    (property "Footprint" "Capacitor_SMD:C_0603_1608Metric" (at 55.88 92.71 0)
+      (effects (font (size 1.27 1.27)) hide)
+    )
+    (property "Datasheet" "~" (at 55.88 92.71 0)
+      (effects (font (size 1.27 1.27)) hide)
+    )
+    (property "LCSC ID" "C14663" (at 55.88 92.71 0)
+      (effects (font (size 1.27 1.27)) hide)
+    )
+    (pin "2")
+    (pin "1")
+    (instances
+      (project "yeg-channel"
+        (path "/edce6e4b-dbee-4006-90c7-70e47f82b9ee/7c2cc44e-c50b-411c-8e87-9b63e86eea9e"
+          (reference "C50") (unit 1)
+        )
+      )
