File: hardware/yeg-channel/yeg-channel.kicad_pcb (KiCad board)
At the start: 2 copper layers, 111 parts, among them J1 Conn_ADC, J2 Conn_Debug, J3 Conn_SPI_Input, J4 Conn_SPI_Output, SW1 SW_RST, SW2 SW_BOOT0, SW3 SW_BOOT1, U1 AMS1117-3.3, U10 HX71708, U11 74HC4051, U2 AMS1117-2.5, U3 LM2664M6X, U4 LM337L_SO8, U5 74HC595, U6 CH32V103C8T6, U7 HX71708, U8 HX71708, U9 HX71708, Y1 32.768k, Y2 8M

Commit message: fixes and add pcb layout
Parts:
- removed D11, D13: D_TVS, Diode_SMD:D_0603_1608Metric
- removed the H1 at (25.4, 30.1)
- removed H5: GND, MountingHole:MountingHole_3.2mm_M3_Pad_TopBottom
- removed the H6 at (33.4, 38.1)
- removed the R13 at (88.9, 67.3)
- removed the R17 at (121.5, 96.0)
- added C51: 100n, Capacitor_SMD:C_0603_1608Metric, F.Cu at (68.5, 43.2)
- added H4: GND, MountingHole:MountingHole_3.2mm_M3_Pad_TopBottom, F.Cu at (127.6, 40.6)
- J2: footprint Connector_PinHeader_2.54mm:PinHeader_1x06_P2.54mm_Vertical -> Connector_PinHeader_2.54mm:PinHeader_1x06_P2.54mm_Horizontal
- R15: value 200 -> 24
- moved H1 106.0 mm to (127.4, 66.9), turned to 180 degrees
- moved D9 99.1 mm to (128.0, 82.0), turned to 180 degrees
- moved D10 94.7 mm to (127.9, 74.2), turned to 180 degrees
- moved D12 94.1 mm to (125.5, 83.4), turned to 90 degrees
- moved J1 90.1 mm to (128.3, 76.8)
- moved H3 88.7 mm to (116.1, 82.8)
- moved R14 80.0 mm to (66.1, 47.2), turned to -90 degrees
- moved Y1 68.4 mm to (76.7, 40.0)
- moved U6 66.4 mm to (86.3, 49.6)
- moved D8 59.5 mm to (91.7, 63.4)
- moved D6 59.0 mm to (96.8, 43.7), turned to 90 degrees
- moved U5 57.8 mm to (109.0, 51.9), turned to 180 degrees
- moved C35 55.4 mm to (77.5, 82.8), turned to 90 degrees
- moved Y2 53.9 mm to (72.5, 51.4), turned to -90 degrees
- moved C36 53.0 mm to (79.0, 82.8), turned to 90 degrees
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- renumbered H2 to H1, H3 to H2, H4 to H3, H7 to H6, R14 to R13, R16 to R14, R18 to R16, R19 to R17, R20 to R18, R21 to R19
Connections:
- C50 pad 1: /ADC/IN+ -> +3V3
- C50 pad 2: /ADC/IN- -> GND
- D12 pad 1: /ADC/SRB1 -> /ADC/SRB2
- D9 pad 1: /ADC/CINA+ -> /ADC/SRB2
- J1 pad 2: /ADC/CINA+ -> /ADC/SRB2
- J2 pad 2: /Connector/UART1_TX -> /Connector/SWDCLK
- J2 pad 3: /Connector/UART1_RX -> /Connector/SWDIO
- J2 pad 4: /Connector/SWDIO -> /Connector/UART1_RX
- J2 pad 5: /Connector/SWDCLK -> /Connector/UART1_TX
- J3 pad 1: /Connector/CS_IN -> /Connector/RCLK
- J3 pad 7: /Connector/RCLK -> /Connector/CS_IN
- J4 pad 1: /Connector/CS_OUT -> /Connector/RCLK
- J4 pad 7: /Connector/RCLK -> /Connector/CS_OUT
- R12 pad 1: /ADC/CINA+ -> /ADC/SRB2
- R15 pad 1: /ADC/SRB1 -> Net-(D6-K)
- R15 pad 2: /ADC/IN- -> GND
Routing:
- net -2V5: track 4.71 -> 195.1 mm, vias 0 -> 7
- net +3V3: track 0.00 -> 140.6 mm, vias 0 -> 2
- net GND: track 1.79 -> 134.1 mm, vias 0 -> 50
- net +2V5: track 0.00 -> 125.4 mm
- net +5V: track 2.73 -> 98.4 mm
- net /ADC/IN-: track 0.00 -> 65.1 mm, vias 0 -> 5
- net /ADC/IN+: track 0.00 -> 59.4 mm, vias 0 -> 5
- net VDDA: track 0.00 -> 57.2 mm
- net /ADC/PD_SCK3: track 0.00 -> 41.5 mm
- net /ADC/PD_SCK2: track 0.00 -> 39.9 mm, vias 0 -> 2
- net /Connector/BOOT1: track 0.00 -> 35.7 mm, vias 0 -> 2
- net /Connector/BOOT0: track 0.00 -> 35.0 mm
- net /MCU/SPI_CS: track 0.00 -> 27.8 mm
- net /ADC/PD_SCK1: track 0.00 -> 26.2 mm, vias 0 -> 2
- net /ADC/SRB2: track 0.00 -> 23.4 mm
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- added copper zone on B.Cu, net GND
- added copper zone on F.Cu, net GND
Other:
- board outline added: 74.9 x 51.4 mm
- board text added: "+5V"
- board text added: "+5V RX TX IO CLK GND"
- board text added: "3V3OK"
- board text added: "5VOK"
- board text added: "ADCOK"
- board text added: "BOOT1 BOOT0"
- board text added: "CINA-"
- board text added: "RST"
- board text added: "SRB2"
- board text added: "SYSOK"
- board text added: "YEG Channel Board by Yet Another AI Ltd Rev.1 Date: Feb. 9th, 2024"
