File: hardware/yeg-channel/yeg-channel.kicad_sch (KiCad schematic)
At the start: 0 parts

Commit message: fixes and add pcb layout
Other:
- title: Yet Another EXG Channel Board -> YEG Channel Board
Changed lines of the file:
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@@
   (paper "A4")
   (title_block
-    (title "Yet Another EXG Channel Board")
+    (title "YEG Channel Board")
     (date "2024-02-07")
     (rev "1")
