File: hardware/yeg-channel/connector.kicad_sch (KiCad schematic)
At the start: 29 parts, among them J1 Conn_ADC, J2 Conn_Debug, J3 Conn_SPI_Input, J4 Conn_SPI_Output, SW1 SW_RST, SW2 SW_BOOT0, SW3 SW_BOOT1

Commit message: fixes and add pcb layout
Parts:
- removed D11, D12: D_TVS, Diode_SMD:D_0603_1608Metric, symbol Device:D_TVS
- removed H1: SRB1, MountingHole:MountingHole_3.2mm_M3_Pad_TopBottom, symbol Mechanical:MountingHole_Pad
- removed H6: GND, MountingHole:MountingHole_3.2mm_M3_Pad_TopBottom, symbol Mechanical:MountingHole_Pad
- added C44: 100n, Capacitor_SMD:C_0603_1608Metric, symbol Device:C_Small
- J2: footprint Connector_PinHeader_2.54mm:PinHeader_1x06_P2.54mm_Vertical -> Connector_PinHeader_2.54mm:PinHeader_1x06_P2.54mm_Horizontal
- renumbered D13 to D12, H2 to H1, H3 to H2, H4 to H3, H5 to H4, H7 to H6
Connections:
- net CINA+ is gone; now on net SRB2: D9.1 (A1), J1.2 (Pin_2)
- net +5V: now also C44.1
- net CS_IN: now also J3.7 (Pin_7); no longer J3.1 (Pin_1)
- net CS_OUT: now also J4.7 (Pin_7); no longer J4.1 (Pin_1)
- net GND: now also C44.2
- net RCLK: now also J3.1 (Pin_1), J4.1 (Pin_1); no longer J3.7 (Pin_7), J4.7 (Pin_7)
- net SWDCLK: now also J2.2 (Pin_2); no longer J2.5 (Pin_5)
- net SWDIO: now also J2.3 (Pin_3); no longer J2.4 (Pin_4)
- net UART1_RX: now also J2.4 (Pin_4); no longer J2.3 (Pin_3)
- net UART1_TX: now also J2.5 (Pin_5); no longer J2.2 (Pin_2)
Other:
- company: (none) -> Yet Another AI Ltd.
- title: (none) -> YEG Channel Board

Commit message: fix bom
Parts:
- J2: LCSC ID C37208 -> C492414
Changed lines of the file:
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@@
       (effects (font (size 1.27 1.27)) hide)
     )
-    (property "LCSC ID" "C37208" (at 22.86 78.74 0)
+    (property "LCSC ID" "C492414" (at 22.86 78.74 0)
       (effects (font (size 1.27 1.27)) hide)
     )
